File: PCB/CarControllerV3/analog.kicad_sch (KiCad schematic)
At the start: 70 parts, among them Q1 BC847B, U1 REF5025AIDGKT, U2 CNY17-2X009T, U20 CD4051BM96, U23 INA241A1IDR, U24 ISO1540, U25 ADS1115IDGS, U3 OPA4188AIDR, U4 CD4051BM96

Commit message: More work to PCB
- Rerouted bunch of connections
- Added alternative charge pump circuit
- Bunch of work on analog circuit
- Removed all the capacitor filter on the connectors in favor of filtering when nessesary.
- Placed canbus on JP5.2, JP5.3
- Disconnected various connections that needs to be decided if we should use.
- Added protection to various areas
- Added various todo notes everywhere..
Parts:
- removed C3, C41, C42, C58: 100n, footprints:CAPC1608X90, symbol CC0603:CC0603KRX7R9BB104
- removed PSU1: DCW03A-12, symbol DCW03:DCW03A-12
- removed R22: 390K, footprints:RC0603FR-RESC1608X60N.pretty, symbol RC0603FR:RC0603FR-07390KL
- removed R24, R51, R52, R53, R54: 1K, footprints:RC0603FR-RESC1608X60N.pretty, symbol RC0603FR:RC0603FR-071KL
- removed R31, R32: 10K, RC0603FR:RC0603FR-RESC1608X60N, symbol RC0603FR:RC0603FR-0710KL
- removed R64: 100R, footprints:RC0603FR-RESC1608X60N.pretty, symbol RC0603FR:RC0603FR-07100R
- removed U1: REF5025AIDGKT, REF5025AIDGKT:REF5025AIDGKT-SOP65P490X110-8N, symbol REF5025AIDGKT:REF5025AIDGKT
- removed U20: CD4051BM96, footprints:SOIC127P600X175-16N, symbol CD4051BM96:CD4051BM96
- removed U3: OPA4188AIDR, footprints:SOIC127P600X175-14N, symbol OPA4188AIDR:OPA4188AIDR
- added C21, C45, C46: 100n, footprints:CAPC1608X90, symbol CC0603:CC0603KRX7R9BB104
- added C22: 10uF, CC0805KKX5R8BB106:CC0805KKX5R8BB106-CAPC2013X145N, symbol CC0805KKX5R8BB106:CC0805KKX5R8BB106
- added D12, D4, D5, D6, D7, D8: 1N4148W-7-F, footprints:1N4148W-7-F-SOD3715X135N, symbol 1N4148W-7-F:1N4148W-7-F
- added IC1: OPA2171AQDRQ1, footprints:OPA2171AQDRQ1-SOIC127P600X175-8N, symbol OPA2171AQDRQ1:OPA2171AQDRQ1
- added R22, R52: 220K, footprints:, symbol RC0603FR:RC0603FR-07220KL
- added R64, R95: 33K, footprints:RC0603FR-RESC1608X60N.pretty, symbol RC0603FR:RC0603FR-0733KL
- added R84, R86, R87: 1K, footprints:RC0603FR-RESC1608X60N.pretty, symbol RC0603FR:RC0603FR-071KL
- added R85, R88, R91, R92, R93: 10K, RC0603FR:RC0603FR-RESC1608X60N, symbol RC0603FR:RC0603FR-0710KL
- added R89: 100R, footprints:RC0603FR-RESC1608X60N, symbol RC0603FR:RC0603FR-07100R
- added R90, R94: 33K, footprints:, symbol RC0603FR:RC0603FR-0733KL
- added U20: AMS1117-3.3, footprints:SOT229P700X180-4N, symbol AMS1117-3.3:AMS1117-3.3
- C69: value 100n -> N.M.; footprint footprints:CAPC1608X90 -> footprints:; symbol CC0603:CC0603KRX7R9BB104 -> CC0603:CC0603_N.M.
Connections:
- net +12v_sense: now also R92.1 (R1)
- net +3V3: now also R37.1 (R1), D12.C, D4.C, D5.C, D7.C; no longer C40.1 (C1), C59.1 (C1), U23.6 (VS), U4.16 (VDD)
- net +5V_1: now also C21.1 (C1), U20.3 (VIN)
- net +HV: now also R52.1 (R1)
- net BAT_MUX_OUT: now also R55.2 (R2)
- net GND: now also C21.2 (C2), C22.1, C45.1 (C1), C46.2 (C2), D6.A, D8.A, IC1.4 (V-), R64.2 (R2), R85.2 (R2), R95.2 (R2), U20.1 (GND/ADJ)
- net GNDA: now also R84.1 (R1)
- net LDR_Senser: now also R91.1 (R1)
- net NTC: now also R93.1 (R1)
- net SHUNT_ANA: now also R86.2 (R2)
- net SPEEDMODE_ANA: now also R90.1 (R1)
- net +3V3_2: now reaches R50.1 (R1), R77.1 (R1), U25.8 (VDD)
- net +3V3_2: now also C40.1 (C1), C59.1 (C1), U23.6 (VS), U4.16 (VDD), C22.2, C45.2 (C2), IC1.8 (V+), R88.1 (R1), U20.2 (VOUT)
- net I2C_SDA_2: now reaches U24.2 (SDA1)
- net I2C_SCL_2: now reaches U24.3 (SCL1)
- net at C60.2 (C2), R55.1 (R1): now also IC1.3 (+IN); no longer U25.4 (AIN0)
- net at R23.1 (R1): now also U25.6 (AIN2), R22.2 (R2)
- net at U25.1 (ADDR): now also R84.2 (R2)
- net at U25.5 (AIN1): now also R86.1 (R1)
- net VREF_VOFFSET: now reaches U25.7 (AIN3)
- net VREF_VOFFSET: now also C69.1 (C1), U23.7 (REF1), R89.1 (R1)
- net SCL_2 renamed I2C_SCL_2_ISO
- net SDA_2 renamed I2C_SDA_2_ISO
- removed net VREF: C69.1 (C1), R37.1 (R1), U23.7 (REF1)
- new net: C46.1 (C1), IC1.5 (+IN), R85.1 (R1), R88.2 (R2)
- new net: IC1.6 (-IN), IC1.7 (OUT), R89.2 (R2)
- new net: R22.1 (R1), R52.2 (R2)
- new net: IC1.1 (OUT), IC1.2 (-IN), R87.2 (R2)
- new net: R87.1 (R1), U25.4 (AIN0)
- new net +12v_sense_ADC: D7.A, D8.C, R92.2 (R2)
- new net LDR_Senser_ADC: D5.A, D6.C, R91.2 (R2)
- new net NTC_ADC: R93.2 (R2)
- new net SPEEDMODE_ANA_ADC: D4.A, R64.1 (R1), R90.2 (R2)
- new net SPEEDOMETER_SIG: R94.1 (R1)
- new net SPEEDOMETER_SIG_ADC: D12.A, R94.2 (R2), R95.1 (R1)
- no-connect marks 1 -> 0
Other:
- note added: "0-5V"
- note added: "0A = 1,65V / 2 = 0,825V"
- note added: "1.65V"
- note added: "MAX -12 to +12V Usually just positive ~150mV"
- note added: "Non-isolated GND"
- note added: "Note: Basically does the same as BAT 1_2 but allows skipping wiring Bat pins Uses different wires on bat for voltage."
- note added: "Note: C69 is risky, can cause Opamp unstability"
- note added: "Offset voltage for Current amplifier"
- note added: "Put in non-isolated ADC These refer the chassis GND / 12V. Would ruin isolation"
- note added: "Uses the internal CMOS protection as reverse protection"
- note added: "VREF ADC = 2.048V"
- note added: "isolated GND"
- note removed: "22-100R"
- note removed: "Note: Divider on connector"
- note removed: "Todo consider REF5040 4.096V"
- note removed: "Todo negative voltage to allow bidirectional?"
- note removed: "Unused!"
- moved on the sheet: C71, C72, C75, C76, C77, C78, C79, L3, PS2, Q1, R23, R50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
