File: PCB/CarControllerV3/connectors2.kicad_sch (KiCad schematic)
At the start: 48 parts, among them J3 649012227222, J4 649012227222, K1 RT424005, K3 RT424005, K4 RT424005, U11 PC817X1NIP1B, U12 PC817X1NIP1B, U15 PC817X1NIP1B, U16 PC817X1NIP1B

Commit message: More work to PCB
- Rerouted bunch of connections
- Added alternative charge pump circuit
- Bunch of work on analog circuit
- Removed all the capacitor filter on the connectors in favor of filtering when nessesary.
- Placed canbus on JP5.2, JP5.3
- Disconnected various connections that needs to be decided if we should use.
- Added protection to various areas
- Added various todo notes everywhere..
Parts:
- removed FL14, FL15, FL16, FL17, FL18: 22nF, footprints:FIL_NFM21CC223R1H3D, symbol NFM21CC223R1H3D:NFM21CC223R1H3D
- added D9: 1N4148W-7-F, footprints:1N4148W-7-F-SOD3715X135N, symbol 1N4148W-7-F:1N4148W-7-F
Connections:
- net +12v_sense: now also D9.A
- net +3V3: now also D9.C
- net Shunt+: now also J3.1, TP35.TP
- net Shunt-: now also J3.2, TP36.TP
Other:
- note added: "Note: already a voltage divider on the ADC sense pin. redo this part"
- note added: "Todo validate IF the shunt + and - is opposite IRL Prior measurements at some point made me remember this might be wrong! OR my car has a fault"
