File: PCB/CarControllerV3/mcu.kicad_sch (KiCad schematic)
At the start: 26 parts, among them IC2 TCAN3404DRBRQ1, J10 Conn_01x02, J12 702471052, K1 RT424005, K2 RT424005, K3 RT424005, K4 RT424005, K5 RT424005, U10 ULN2003APW, U18 STM32C092RCT6, Y1 16MHz

Commit message: More work to PCB
- Rerouted bunch of connections
- Added alternative charge pump circuit
- Bunch of work on analog circuit
- Removed all the capacitor filter on the connectors in favor of filtering when nessesary.
- Placed canbus on JP5.2, JP5.3
- Disconnected various connections that needs to be decided if we should use.
- Added protection to various areas
- Added various todo notes everywhere..
Parts:
- removed J12: 702471052, footprints:CONN_7024710XX_MOL, symbol 702471052:702471052
- added C26: 4.7uF, footprints:CC0402-CAPC1005X55N, symbol CC0402:CC0402MRX5R5BB475
- added J14: 2x5, 61201021621:61201021621, symbol 6120XX21621_61201021621:6120XX21621_61201021621
- added R24: 100R, footprints:RC0603FR-RESC1608X60N, symbol RC0603FR:RC0603FR-07100R
Connections:
- net +3V3: now also C26.2 (C2), R24.1 (R1)
- net CHARGER_STOP_SIG: now also U18.42 (PA10); no longer U18.61 (PB7)
- net GND: now also C26.1 (C1), J14.5, J14.6
- net IGNITION_ON: now also U18.37 (PA9); no longer U18.60 (PB6)
- net K1_SIG: now also U18.52 (PD2); no longer U18.31 (PB11)
- net K2_SIG: now also U18.53 (PD3); no longer U18.32 (PB12)
- net K3_SIG: now also U18.54 (PD4); no longer U18.33 (PB13)
- net K4_SIG: now also U18.55 (PD5); no longer U18.34 (PB14)
- net K5_SIG: now also U18.56 (PD6); no longer U18.35 (PB15)
- net MCU_RST: now also J14.1
- net SWDCLK_BOOT0: now also J14.2
- net SWDIO: now also J14.4
- net SPEEDMODE_ANA_ADC: now reaches U18.17 (PA0)
- net LDR_Senser_ADC: now reaches U18.18 (PA1)
- net NTC_ADC: now reaches U18.19 (PA2)
- net SPEEDOMETER_SIG_ADC: now reaches U18.20 (PA3)
- net MCU_PWM_CHG_PMP: now reaches U18.4 (PC14-OSCX_IN)
- net UART_RX renamed I2C_SDA_2
- net UART_TX renamed I2C_SCL_2
- new net: J14.7, J14.8, R24.2 (R2)
- new net I2C_SCL_1: U18.35 (PB15)
- new net I2C_SDA_1: U18.34 (PB14)
- new net UART_MCU_RX: U18.60 (PB6)
- new net UART_MCU_TX: U18.61 (PB7)
Other:
- note added: "ADC"
- note removed: "+3.3V +5.0V"
- note removed: "2x5 IDE Compatible with ST-link v2 Expects 1-1 cable"
- note removed: "SWIM"
- note removed: "WRONG HEADER!! It is a IDE header"
- moved on the sheet: J10, R34, R63, S1
